File: PLC4UNIPCB/OUT-RELAY-1.kicad_sch (KiCad schematic)
At the start: 7 parts, among them K1 Fujitsu_FTR-LYCA005x, Q10 BFN26

Commit message: Add files via upload
Parts:
- removed K1: Fujitsu_FTR-LYCA005x, Relay_THT:Relay_SPDT_Fujitsu_FTR-LYCA005x_FormC_Vertical, symbol Relay:Fujitsu_FTR-LYCA005x
- removed OC7: FOD817S, Package_DIP_AKL:SMDIP-4_W9.53mm, symbol Optocoupler_AKL:FOD817S
- removed Q10: BFN26, Package_TO_SOT_SMD_AKL:SOT-23, symbol Transistor_BJT_AKL:BFN26
- removed R33: 510, Resistor_SMD_AKL:R_0603_1608Metric, symbol Resistor_AKL:R_0603
- removed R34: 2K, Resistor_SMD_AKL:R_0603_1608Metric, symbol Resistor_AKL:R_0603
- removed R35: 10K, Resistor_SMD_AKL:R_0603_1608Metric, symbol Resistor_AKL:R_0603
- added K1: G5V-1, Relay_THT:Relay_SPDT_Omron_G5V-1, symbol Relay:G5V-1
- added Q7: BC817, PCM_Package_TO_SOT_SMD_AKL:SOT-23, symbol PCM_Transistor_BJT_AKL:BC817
- added R35: 2.4k, PCM_Resistor_SMD_AKL:R_0603_1608Metric, symbol GP8211S-TC50:R_0603
- renumbered D2 to D5
Connections:
- net GND: now also Q7.2 (E)
- net IN: now also R35.1
- net VCC: now also K1.2
- net out-common-1: now also K1.5, K1.6
- net out-nc: now also K1.1
- net out-no-1: now also K1.10
- net at D5.2 (A): now also K1.9, Q7.3 (C)
- new net: Q7.1 (B), R35.2
