File: PLC4UNIPCB/OUT-RELAY-2.kicad_sch (KiCad schematic)
At the start: 7 parts, among them K2 Fujitsu_FTR-LYAA005x, Q11 BFN26

Commit message: Add files via upload
Parts:
- removed R36: 2K, Resistor_SMD_AKL:R_0603_1608Metric, symbol Resistor_AKL:R_0603
- removed R37: 10K, Resistor_SMD_AKL:R_0603_1608Metric, symbol Resistor_AKL:R_0603
- removed R38: 510, Resistor_SMD_AKL:R_0603_1608Metric, symbol Resistor_AKL:R_0603
- added R33: 510, PCM_Resistor_SMD_AKL:R_0603_1608Metric, symbol GP8211S-TC50:R_0603
- added R34: 2K, PCM_Resistor_SMD_AKL:R_0603_1608Metric, symbol GP8211S-TC50:R_0603
- added R35: 10K, PCM_Resistor_SMD_AKL:R_0603_1608Metric, symbol GP8211S-TC50:R_0603
- Q7: renamed from Q11; LCSC (none) -> C39828
- renumbered D3 to D7, OC8 to OC5
Connections:
- net GND: now also R34.1
- net IN: now also R33.1
- net at OC5.1: now also R33.2
- net at OC5.3: now also R34.2, R35.1
- net at Q7.1 (B): now also R35.2
