File: PLC4UNIPCB/Out_npn.kicad_sch (KiCad schematic)
At the start: 3 parts

Commit message: Add files via upload
Parts:
- removed Q?: BFN26, Package_TO_SOT_SMD_AKL:SOT-23, symbol Transistor_BJT_AKL:BFN26
- removed R? (x2): 2.4k, Resistor_SMD_AKL:R_0603_1608Metric, symbol Resistor_AKL:R_0603
- added Q5: BC817, PCM_Package_TO_SOT_SMD_AKL:SOT-23, symbol PCM_Transistor_BJT_AKL:BC817
- added R30: 2.4k, PCM_Resistor_SMD_AKL:R_0603_1608Metric, symbol GP8211S-TC50:R_0603
- added R31: 10k, PCM_Resistor_SMD_AKL:R_0603_1608Metric, symbol GP8211S-TC50:R_0603
Connections:
- net GND: now also Q5.2 (E), R31.1
- net IN: now also R30.1
- net OUT: now also Q5.3 (C)
- new net: Q5.1 (B), R30.2, R31.2
