File: PLC4UNIPCB/Output_0-10V.kicad_sch (KiCad schematic)
At the start: 6 parts

Commit message: Add files via upload
Parts:
- removed R17, R18: 4.7k, PCM_SparkFun-Resistor:R_0603_1608Metric, symbol PCM_SparkFun-Resistor:4.7k_0603
- added R14, R15: 4.7k, PCM_Resistor_SMD_AKL:R_0603_1608Metric, symbol GP8211S-TC50:R_0603
- renumbered C1 to C3, C2 to C4, D2 to D1, U2 to U4
Connections:
- net +3.3V: now also R14.1, R15.1
- net SCL: now also R14.2
- net SDA: now also R15.2
- net +12V renamed VCC
