File: PLC4UNIPCB/input-npn-opto.kicad_sch (KiCad schematic)
At the start: 3 parts

Commit message: Add files via upload
Parts:
- removed OC?: FOD817S, Package_DIP_AKL:SMDIP-4_W9.53mm, symbol Optocoupler_AKL:FOD817S
- removed R? (x2): 2.4K, PCM_Resistor_SMD_AKL:R_0603_1608Metric, symbol GP8211S-TC50:R_0603
- added OC1: TLP293, PCM_Package_SO_AKL:SOP-4_4.4x2.6mm_P1.27mm, symbol PCM_Optocoupler_AKL:TLP293
- added R6, R7: 10K, PCM_Resistor_SMD_AKL:R_0603_1608Metric, symbol GP8211S-TC50:R_0603
Connections:
- net +3.3V: now also R7.1
- net GND: now also OC1.3
- net IN: now also OC1.2
- net OUT: now also OC1.4, R7.2
- net VCC: now also R6.1
- new net: OC1.1, R6.2
