File: PLC4UNIPCB/input-pnp-opto.kicad_sch (KiCad schematic)
At the start: 3 parts

Commit message: Add files via upload
Parts:
- removed OC?: FOD817S, Package_DIP_AKL:SMDIP-4_W9.53mm, symbol Optocoupler_AKL:FOD817S
- added OC2: TLP293, PCM_Package_SO_AKL:SOP-4_4.4x2.6mm_P1.27mm, symbol PCM_Optocoupler_AKL:TLP293
- R8: renamed from R?; value 2.4K -> 4.7K
- gave numbers to parts that had none: 1
Connections:
- net GND: now also OC2.2, OC2.3
- net OUT: now also OC2.4
- net at R8.2: now also OC2.1
Changed lines of the file:
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@@
 		(on_board yes)
 		(dnp no)
-		(property "Reference" "R?"
+		(property "Reference" "R8"
 			(at 114.3001 99.06 0)
 			(effects
@@
 			)
 		)
-		(property "Value" "2.4K"
+		(property "Value" "4.7K"
 			(at 111.7601 99.06 0)
 			(effects
@@
 			(project "PLC4UNIPCB"
 				(path "/20dd9fa8-33e5-4e01-8b4a-8cb5828152c9/ef44eee8-cd41-4527-92e2-6c408c0d0d91/7d73415a-6d92-4775-9fde-5e791787ec39"
-					(reference "R?")
-					(unit 1)
-				)
-				(path "/20dd9fa8-33e5-4e01-8b4a-8cb5828152c9/ef44eee8-cd41-4527-92e2-6c408c0d0d91/993499e7-3317-45fe-8d12-a8e3207aa57a"
-					(reference "R?")
+					(reference "R8")
+					(unit 1)
+				)
+				(path "/20dd9fa8-33e5-4e01-8b4a-8cb5828152c9/ef44eee8-cd41-4527-92e2-6c408c0d0d91/993499e7-3317-45fe-8d12-a8e3207aa57a"
+					(reference "R23")
 					(unit 1)
 				)
@@
 		(on_board yes)
 		(dnp no)
-		(property "Reference" "R?"
+		(property "Reference" "R9"
 			(at 125.73 96.5199 0)
 			(effects
@@
 			(project "PLC4UNIPCB"
 				(path "/20dd9fa8-33e5-4e01-8b4a-8cb5828152c9/ef44eee8-cd41-4527-92e2-6c408c0d0d91/7d73415a-6d92-4775-9fde-5e791787ec39"
-					(reference "R?")
-					(unit 1)
-				)
-				(path "/20dd9fa8-33e5-4e01-8b4a-8cb5828152c9/ef44eee8-cd41-4527-92e2-6c408c0d0d91/993499e7-3317-45fe-8d12-a8e3207aa57a"
-					(reference "R11")
+					(reference "R9")
+					(unit 1)
+				)
+				(path "/20dd9fa8-33e5-4e01-8b4a-8cb5828152c9/ef44eee8-cd41-4527-92e2-6c408c0d0d91/993499e7-3317-45fe-8d12-a8e3207aa57a"
+					(reference "R24")
 					(unit 1)
 				)
@@
 		(dnp no)
 		(fields_autoplaced yes)
-		(property "Reference" "#PWR06"
+		(property "Reference" "#PWR013"
 			(at 120.65 127 0)
 			(effects
@@
 			(project "PLC4UNIPCB"
 				(path "/20dd9fa8-33e5-4e01-8b4a-8cb5828152c9/ef44eee8-cd41-4527-92e2-6c408c0d0d91/7d73415a-6d92-4775-9fde-5e791787ec39"
-					(reference "#PWR06")
+					(reference "#PWR013")
+					(unit 1)
+				)
+				(path "/20dd9fa8-33e5-4e01-8b4a-8cb5828152c9/ef44eee8-cd41-4527-92e2-6c408c0d0d91/993499e7-3317-45fe-8d12-a8e3207aa57a"
+					(reference "#PWR042")
 					(unit 1)
 				)
@@
 	)
 	(symbol
-		(lib_id "Optocoupler_AKL:FOD817S")
+		(lib_id "PCM_Optocoupler_AKL:TLP293")
 		(at 124.46 113.03 0)
 		(unit 1)
@@
 		(on_board yes)
 		(dnp no)
-		(property "Reference" "OC?"
+		(fields_autoplaced yes)
+		(property "Reference" "OC2"
 			(at 132.08 111.7599 0)
 			(effects
@@
 			)
 		)
-		(property "Value" "FOD817S"
+		(property "Value" "TLP293"
 			(at 132.08 114.2999 0)
 			(effects
@@
 				)
 				(justify left)
-				(hide yes)
-			)
-		)
-		(property "Footprint" "Package_DIP_AKL:SMDIP-4_W9.53mm"
-			(at 119.38 118.11 0)
+			)
+		)
+		(property "Footprint" "PCM_Package_SO_AKL:SOP-4_4.4x2.6mm_P1.27mm"
+			(at 130.81 111.76 0)
 			(effects
 				(font
@@
 			)
 		)
-		(property "Datasheet" "https://www.tme.eu/Document/3a0358906a5fcb3aa253d025de809a1d/FOD814300W.PDF"
+		(property "Datasheet" "https://www.tme.eu/Document/4529df8a9c1b6d8255594aba717bca36/TLP293-E-T.pdf"
 			(at 124.46 113.03 0)
 			(effects
@@
 			)
 		)
-		(property "Description" "SMDIP-4 Optocoupler, Transistor output, 5kV, 8us, Alternate KiCAD Library"
+		(property "Description" "SO-4 Optocoupler, Transistor output, 3.75kV, 3us, Alternate KiCAD Library"
 			(at 124.46 113.03 0)
 			(effects
@@
 			)
 		)
-		(property "Part Number" "LTV-354"
-			(at 134.874 114.3 0)
-			(effects
-				(font
-					(size 1.27 1.27)
-				)
-			)
+		(pin "1"
 		)
 		(pin "3"
 		)
+		(pin "2"
+		)
 		(pin "4"
 		)
-		(pin "2"
-		)
-		(pin "1"
-		)
-		(instances
-			(project "PLC4UNIPCB"
-				(path "/20dd9fa8-33e5-4e01-8b4a-8cb5828152c9/ef44eee8-cd41-4527-92e2-6c408c0d0d91/7d73415a-6d92-4775-9fde-5e791787ec39"
-					(reference "OC?")
+		(instances
+			(project "PLC4UNIPCB"
+				(path "/20dd9fa8-33e5-4e01-8b4a-8cb5828152c9/ef44eee8-cd41-4527-92e2-6c408c0d0d91/7d73415a-6d92-4775-9fde-5e791787ec39"
+					(reference "OC2")
+					(unit 1)
+				)
+				(path "/20dd9fa8-33e5-4e01-8b4a-8cb5828152c9/ef44eee8-cd41-4527-92e2-6c408c0d0d91/993499e7-3317-45fe-8d12-a8e3207aa57a"
+					(reference "OC4")
 					(unit 1)
 				)
@@
 		(dnp no)
 		(fields_autoplaced yes)
-		(property "Reference" "#PWR08"
+		(property "Reference" "#PWR014"
 			(at 128.27 96.52 0)
 			(effects
@@
 			(project "PLC4UNIPCB"
 				(path "/20dd9fa8-33e5-4e01-8b4a-8cb5828152c9/ef44eee8-cd41-4527-92e2-6c408c0d0d91/7d73415a-6d92-4775-9fde-5e791787ec39"
-					(reference "#PWR08")
+					(reference "#PWR014")
+					(unit 1)
+				)
+				(path "/20dd9fa8-33e5-4e01-8b4a-8cb5828152c9/ef44eee8-cd41-4527-92e2-6c408c0d0d91/993499e7-3317-45fe-8d12-a8e3207aa57a"
+					(reference "#PWR043")
 					(unit 1)
 				)
@@
 		(dnp no)
 		(fields_autoplaced yes)
-		(property "Reference" "#PWR010"
+		(property "Reference" "#PWR015"
 			(at 128.27 127 0)
 			(effects
@@
 			(project "PLC4UNIPCB"
 				(path "/20dd9fa8-33e5-4e01-8b4a-8cb5828152c9/ef44eee8-cd41-4527-92e2-6c408c0d0d91/7d73415a-6d92-4775-9fde-5e791787ec39"
-					(reference "#PWR010")
-					(unit 1)
-				)
+					(reference "#PWR015")
+					(unit 1)
+				)
+				(path "/20dd9fa8-33e5-4e01-8b4a-8cb5828152c9/ef44eee8-cd41-4527-92e2-6c408c0d0d91/993499e7-3317-45fe-8d12-a8e3207aa57a"
+					(reference "#PWR044")
+					(unit 1)
+				)
