File: PLC4UNIPCB/output-pnp.kicad_sch (KiCad schematic)
At the start: 3 parts

Commit message: Add files via upload
Parts:
- removed Q?: 2SA2018, Package_TO_SOT_SMD_AKL:SOT-416, symbol Transistor_BJT_AKL:2SA2018
- removed R? (x2): 2.4k, Resistor_SMD_AKL:R_0603_1608Metric, symbol Resistor_AKL:R_0603
- added D7: M7, PCM_Diode_SMD_AKL:D_SMA, symbol PCM_Diode_AKL:M7
- added Q10: BC817, PCM_Package_TO_SOT_SMD_AKL:SOT-23, symbol PCM_Transistor_BJT_AKL:BC817
- added Q11: MMBT4403, PCM_Package_TO_SOT_SMD_AKL:SOT-23, symbol PCM_Transistor_BJT_AKL:MMBT4403
- added R39: 2.4k, PCM_Resistor_SMD_AKL:R_0603_1608Metric, symbol GP8211S-TC50:R_0603
- added R40, R42, R43: 10k, PCM_Resistor_SMD_AKL:R_0603_1608Metric, symbol GP8211S-TC50:R_0603
- added R41: 4.7k, PCM_Resistor_SMD_AKL:R_0603_1608Metric, symbol GP8211S-TC50:R_0603
Connections:
- net GND: now also D7.2 (A), Q10.2 (E), R40.1, R43.1
- net IN: now also R39.1
- net OUT: now also D7.1 (K), Q11.3 (C), R43.2
- net VCC: now also Q11.2 (E), R41.2
- new net: Q10.1 (B), R39.2, R40.2
- new net: Q10.3 (C), R41.1, R42.1
- new net: Q11.1 (B), R42.2
