File: PLC4UNIPCB/Board-PLC4UNI-G1W.kicad_sch (KiCad schematic)
At the start: 0 parts

Commit message: Add files via upload
Other:
- removed sheet CT
- removed sheet VAC
- added sheet SourceProtection (source protection.kicad_sch)
- sheet Input_4-20mA ports: added none; removed IN_4-20mA, IN_4-20mA_2
- sheet Input_NPN1_Opto ports: added IN, OUT; removed In-, Out
- sheet Input_NPN1_Opto1 ports: added IN, OUT; removed In-, Out
- sheet Input_PNP1_Opto ports: added IN, OUT; removed In+, Out
- sheet Input_PNP2_Opto ports: added IN, OUT; removed In+, Out
- sheet OutRelay2: file OUT-RELAY-2.kicad_sch -> OUT-RELAY-1.kicad_sch
- sheet OutRelay2 ports: added out-common-1, out-nc, out-no-1; removed out-common-2, out-no-2
- sheet Output_4-20mA: file Output_4-20mA.kicad_sch -> mA_INTERFAZ.kicad_sch
- sheet Output_4-20mA ports: added SCLK, SDA, mA_OUT+; removed Out_4-20mA
- sheet Output_4-20mA1: file Output_4-20mA.kicad_sch -> mA_INTERFAZ.kicad_sch
- sheet Output_4-20mA1 ports: added SCLK, SDA, mA_OUT+; removed Out_4-20mA
- sheet PLC4UNI ports: added IN_4-20mA, IN_4-20mA_2; removed Out_4-20mA
- sheet RS485_Module1_protect: file RS485_Module1_protect.kicad_sch -> RS485 (2).kicad_sch
- sheet RS485_Module1_protect ports: added RS-485 A, RS-485 B, UART_RX, UART_TX, ~{TX}/RX; removed Con, Din, Dout, con-a, con-b

Commit message: Add files via upload
Other:
- sheet PLC4UNI ports: added Out_4-20mA, USB+, USB-; removed none
Changed lines of the file:
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@@
+	(wire
+		(pts
+			(xy 104.14 72.39) (xy 129.54 72.39)
+		)
+		(stroke
+			(width 0)
+			(type default)
+		)
+	)
 	(wire
 		(pts
@@
 		(pts
 			(xy 166.37 20.32) (xy 170.18 20.32)
+		)
+		(stroke
+			(width 0)
+			(type default)
+		)
+	)
+	(wire
+		(pts
+			(xy 104.14 74.93) (xy 129.54 74.93)
 		)
 		(stroke
@@
 		)
 	)
+	(hierarchical_label "USB+"
+		(shape input)
+		(at 104.14 72.39 180)
+		(effects
+			(font
+				(size 1.27 1.27)
+			)
+			(justify right)
+		)
+	)
 	(hierarchical_label "NPN_OUT1"
 		(shape output)
@@
 			)
 			(justify left)
+		)
+	)
+	(hierarchical_label "USB-"
+		(shape input)
+		(at 104.14 74.93 180)
+		(effects
+			(font
+				(size 1.27 1.27)
+			)
+			(justify right)
 		)
 	)
@@
 			(effects
 				(font
+					(size 1.27 1.27)
+				)
+				(justify left)
+			)
+		)
+		(pin "Out_4-20mA" output
+			(at 166.37 38.1 0)
+			(effects
+				(font
+					(size 1.27 1.27)
+				)
+				(justify right)
+			)
+		)
+		(pin "USB+" input
+			(at 129.54 72.39 180)
+			(effects
+				(font
+					(size 1.27 1.27)
+				)
+				(justify left)
+			)
+		)
+		(pin "USB-" input
+			(at 129.54 74.93 180)
+			(effects
+				(font
