File: PLC4UNIPCB/CPU.kicad_sch (KiCad schematic)
At the start: 1 part, among them U1 ESP32-S3-DevKitC

Commit message: Add files via upload
Parts:
- removed U1: ESP32-S3-DevKitC, PCM_Espressif:ESP32-S3-DevKitC, symbol GP8211S-TC50:ESP32-S3-DevKitC
- added H1, H2: MountingHole_M3, MountingHole:MountingHole_3.2mm_M3, symbol PCM_SL_Mechanical:MountingHole_M3
- added R4, R5: 10k, PCM_Resistor_SMD_AKL:R_0603_1608Metric, symbol GP8211S-TC50:R_0603
- added U8: ESP32-S3-MINI-1U, RF_Module:ESP32-S2-MINI-1U, symbol RF_Module:ESP32-S3-MINI-1U
Connections:
- net +3.3V: now also R4.1, R5.1, U8.3 (3V3)
- net GND: now also U8.1 (GND), U8.2 (GND), U8.42 (GND), U8.43 (GND), U8.46 (GND), U8.47 (GND), U8.48 (GND), U8.49 (GND), U8.50 (GND), U8.51 (GND), U8.52 (GND), U8.53 (GND), U8.54 (GND), U8.55 (GND), U8.56 (GND), U8.57 (GND), U8.58 (GND), U8.59 (GND), U8.60 (GND), U8.61 (GND), U8.62 (GND), U8.63 (GND), U8.64 (GND), U8.65 (GND)
- net SCL: now also R4.2
- net SDA: now also R5.2
- net micro_rs485_rx: now also U8.40 (RXD0)
- net micro_rs485_tx: now also U8.39 (TXD0)

Commit message: Add files via upload
Parts:
- removed R4, R5: 10k, PCM_Resistor_SMD_AKL:R_0603_1608Metric, symbol GP8211S-TC50:R_0603
- added J5: USB_C_Receptacle, PCM_SparkFun-Connector:USB-C_16, symbol PCM_SparkFun-Connector:USB_C_Receptacle
Connections:
- net GND: now also J5.GND
- net IN_4-20mA: now also U8.7 (IO3)
- net IN_4-20mA_2: now also U8.8 (IO4)
- net IN_NPN: now also U8.26 (IO26)
- net IN_NPN1_Opto: now also U8.31 (IO35)
- net IN_NPN2: now also U8.25 (IO21)
- net IN_NPN2_Opto: now also U8.32 (IO36)
- net IN_PNP1: now also U8.34 (IO38)
- net IN_PNP1_Opto: now also U8.28 (IO33)
- net IN_PNP2: now also U8.33 (IO37)
- net IN_PNP2_Opto: now also U8.29 (IO34)
- net NPN_OUT1: now also U8.5 (IO1)
- net NPN_OUT2: now also U8.4 (IO0)
- net OUT_RELAY1: now also U8.30 (IO48)
- net OUT_RELAY2: now also U8.6 (IO2)
- net Opto_NPN: now also U8.44 (IO46)
- net Opto_NPN2: now also U8.27 (IO47)
- net Out_4-20mA: now also U8.35 (IO39)
- net Out_4-20mA_2: now also U8.36 (IO40)
- net PNP_OUT1: now also U8.37 (IO41)
- net PNP_OUT2: now also U8.38 (IO42)
- net PNP_OUT3: now also U8.41 (IO45)
- net SCL: now also U8.13 (IO9)
- net SDA: now also U8.12 (IO8)
- net USB+: now also U8.24 (USB_D+), J5.A6 (D+), J5.B6 (D+)
- net USB-: now also U8.23 (USB_D-), J5.A7 (D-), J5.B7 (D-)
- net micro1_rs485_control: now also U8.9 (IO5)
