File: PLC4UNIPCB/PLC4UNIPCB.kicad_pcb (KiCad board)
At the start: 2 copper layers, 2 parts

Commit message: Add files via upload
Actualización de Esquemáticos
Parts:
- added D1: SM712, PCM_Package_TO_SOT_SMD_AKL:SOT-23, F.Cu at (84.7, 71.1)
- added J1: NPN_IN, TerminalBlock_Phoenix:TerminalBlock_Phoenix_PT-1,5-4-3.5-H_1x04_P3.50mm_Horizontal, F.Cu at (18.9, 103.0)
- added J2: PNP_IN, TerminalBlock_Phoenix:TerminalBlock_Phoenix_PT-1,5-4-3.5-H_1x04_P3.50mm_Horizontal, F.Cu at (18.9, 113.0)
- added J3: RS485, TerminalBlock_Phoenix:TerminalBlock_Phoenix_PT-1,5-3-3.5-H_1x03_P3.50mm_Horizontal, F.Cu at (34.9, 103.0)
- added J4: NPN_Out, TerminalBlock_Phoenix:TerminalBlock_Phoenix_PT-1,5-4-3.5-H_1x04_P3.50mm_Horizontal, F.Cu at (18.9, 122.9)
- added J5: PNP_Out, TerminalBlock_Phoenix:TerminalBlock_Phoenix_PT-1,5-3-3.5-H_1x03_P3.50mm_Horizontal, F.Cu at (34.9, 113.0)
- added J6: 4-20mA_Out, TerminalBlock_Phoenix:TerminalBlock_Phoenix_PT-1,5-2-3.5-H_1x02_P3.50mm_Horizontal, F.Cu at (34.9, 122.9)
- added OC1: FOD817S, PCM_Package_DIP_AKL:SMDIP-4_W9.53mm, F.Cu at (83.6, 116.3)
- added OC2: FOD817S, PCM_Package_DIP_AKL:SMDIP-4_W9.53mm, F.Cu at (68.4, 102.2)
- added OC3: FOD817S, PCM_Package_DIP_AKL:SMDIP-4_W9.53mm, F.Cu at (73.7, 72.1)
- added OC4: FOD817S, PCM_Package_DIP_AKL:SMDIP-4_W9.53mm, F.Cu at (68.4, 116.3)
- added OC5: FOD817S, PCM_Package_DIP_AKL:SMDIP-4_W9.53mm, F.Cu at (73.7, 58.0)
- added OC6: FOD817S, PCM_Package_DIP_AKL:SMDIP-4_W9.53mm, F.Cu at (53.3, 102.2)
- added OC7: FOD817S, PCM_Package_DIP_AKL:SMDIP-4_W9.53mm, F.Cu at (83.6, 102.2)
- added OC8: FOD817S, PCM_Package_DIP_AKL:SMDIP-4_W9.53mm, F.Cu at (53.3, 116.3)
- added R1: 2.4K, PCM_Resistor_SMD_AKL:R_0603_1608Metric, F.Cu at (63.9, 106.9)
- added R10: 2.4K, PCM_Resistor_SMD_AKL:R_0603_1608Metric, F.Cu at (48.8, 109.6)
- added R11: 2.4K, PCM_Resistor_SMD_AKL:R_0603_1608Metric, F.Cu at (69.2, 79.5)
- added R12: 2.4K, PCM_Resistor_SMD_AKL:R_0603_1608Metric, F.Cu at (79.1, 123.7)
- added R13: 2.4K, PCM_Resistor_SMD_AKL:R_0603_1608Metric, F.Cu at (79.1, 106.9)
- added R14: 2.4K, PCM_Resistor_SMD_AKL:R_0603_1608Metric, F.Cu at (79.1, 109.6)
- added R15: 2.4K, PCM_Resistor_SMD_AKL:R_0603_1608Metric, F.Cu at (48.8, 121.0)
- added R16: 2.4K, PCM_Resistor_SMD_AKL:R_0603_1608Metric, F.Cu at (48.8, 123.7)
- added R2: 2.4K, PCM_Resistor_SMD_AKL:R_0603_1608Metric, F.Cu at (63.9, 121.0)
- added R3: 2.4K, PCM_Resistor_SMD_AKL:R_0603_1608Metric, F.Cu at (63.9, 123.7)
- added R4: 2.4K, PCM_Resistor_SMD_AKL:R_0603_1608Metric, F.Cu at (79.1, 121.0)
- added R5: 2.4K, PCM_Resistor_SMD_AKL:R_0603_1608Metric, F.Cu at (63.9, 109.6)
- added R6: 2.4K, PCM_Resistor_SMD_AKL:R_0603_1608Metric, F.Cu at (69.2, 76.8)
- added R7: 2.4K, PCM_Resistor_SMD_AKL:R_0603_1608Metric, F.Cu at (69.2, 62.7)
- added R8: 2.4K, PCM_Resistor_SMD_AKL:R_0603_1608Metric, F.Cu at (69.2, 65.4)
- added R9: 2.4K, PCM_Resistor_SMD_AKL:R_0603_1608Metric, F.Cu at (48.8, 106.9)
- added U1: ESP32-S3-WROOM-1, RF_Module:ESP32-S3-WROOM-1, F.Cu at (40.6, 82.9)

Commit message: Add files via upload
Parts:
- removed J5: PNP_Out, TerminalBlock_Phoenix:TerminalBlock_Phoenix_PT-1,5-3-3.5-H_1x03_P3.50mm_Horizontal
- removed J6: 4-20mA_Out, TerminalBlock_Phoenix:TerminalBlock_Phoenix_PT-1,5-2-3.5-H_1x02_P3.50mm_Horizontal
- removed OC5, OC6, OC7, OC8: FOD817S, PCM_Package_DIP_AKL:SMDIP-4_W9.53mm
- removed REF** (x2): MountingHole_2.5mm, MountingHole:MountingHole_2.5mm
- added C1: 100nF, Capacitor_SMD:C_0201_0603Metric, F.Cu at (51.1, 111.1)
- added C10: 1uF, Capacitor_SMD:C_0805_2012Metric, F.Cu at (40.4, 89.3)
- added C11: 10uF, PCM_Capacitor_SMD_AKL:C_1206_3216Metric, F.Cu at (138.0, 76.5)
- added C12: 100nF, PCM_Capacitor_SMD_AKL:C_0805_2012Metric, F.Cu at (146.2, 71.8)
- added C13: 22uF, PCM_Capacitor_SMD_AKL:C_1206_3216Metric, F.Cu at (142.0, 80.8)
- added C14: 22uF, PCM_Capacitor_SMD_AKL:C_1206_3216Metric, F.Cu at (142.0, 78.0)
- added C2: 0.1uF, PCM_Capacitor_SMD_AKL:C_0603_1608Metric, F.Cu at (182.7, 73.7)
- added C3: 1uF, PCM_Capacitor_SMD_AKL:C_0603_1608Metric, F.Cu at (210.7, 124.8)
- added C4: 0.1uF, PCM_Capacitor_SMD_AKL:C_0603_1608Metric, F.Cu at (207.4, 125.5)
- added C5: 220pF, Capacitor_SMD:C_0805_2012Metric, F.Cu at (40.4, 99.2)
- added C6: 1uF, Capacitor_SMD:C_0805_2012Metric, F.Cu at (40.4, 102.3)
- added C7: 1uF, Capacitor_SMD:C_0805_2012Metric, F.Cu at (40.4, 105.3)
- added C8: 220pF, Capacitor_SMD:C_0805_2012Metric, F.Cu at (40.4, 83.3)
- added C9: 1uF, Capacitor_SMD:C_0805_2012Metric, F.Cu at (40.4, 86.3)
- added D10: D_Zener, Diode_SMD:D_0603_1608Metric, F.Cu at (48.7, 92.9)
- added D11: SMF24A, Diode_SMD:D_SMF, F.Cu at (49.5, 89.9)
- added D2: D_Zener, Diode_SMD:D_0603_1608Metric, F.Cu at (48.7, 108.8)
- added D3: SMF24A, Diode_SMD:D_SMF, F.Cu at (49.5, 105.9)
- added D5: 1N4148WT, Diode_SMD:D_SOD-523, F.Cu at (175.8, 123.0)
- added D6: 1N4148WT, Diode_SMD:D_SOD-523, F.Cu at (185.9, 122.6)
- added D7: M7, PCM_Diode_SMD_AKL:D_SMA, F.Cu at (162.6, 125.3)
- added D8: M7, PCM_Diode_SMD_AKL:D_SMA, F.Cu at (154.4, 125.8)
- added D9: M7, PCM_Diode_SMD_AKL:D_SMA, F.Cu at (171.5, 125.6)
- added F1: Fuse, Fuse:Fuse_1812_4532Metric, F.Cu at (137.8, 70.0)
- added H1: MountingHole_M3, MountingHole:MountingHole_3.2mm_M3, F.Cu at (226.5, 73.2)
- added H2: MountingHole_M3, MountingHole:MountingHole_3.2mm_M3, F.Cu at (141.5, 123.2)
- added K1: G5V-1, Relay_THT:Relay_SPDT_Omron_G5V-1, F.Cu at (178.3, 117.9)
- added K2: G5V-1, Relay_THT:Relay_SPDT_Omron_G5V-1, F.Cu at (188.4, 117.8)
- added L1: ANR4030T6R8M, Inductor_SMD:L_APV_ANR4030, F.Cu at (147.0, 75.5)
- added LED1: LED_0603_Red, PCM_LED_SMD_AKL:LED_0603_1608Metric, F.Cu at (135.2, 61.7)
- added Q10: BC817, PCM_Package_TO_SOT_SMD_AKL:SOT-23, F.Cu at (162.6, 117.6)
- added Q11: MMBT4403, PCM_Package_TO_SOT_SMD_AKL:SOT-23, F.Cu at (158.6, 124.8)
- added Q12: BC817, PCM_Package_TO_SOT_SMD_AKL:SOT-23, F.Cu at (154.3, 118.0)
- added Q13: MMBT4403, PCM_Package_TO_SOT_SMD_AKL:SOT-23, F.Cu at (149.4, 124.5)
- added Q14: BC817, PCM_Package_TO_SOT_SMD_AKL:SOT-23, F.Cu at (171.4, 118.0)
- added Q15: MMBT4403, PCM_Package_TO_SOT_SMD_AKL:SOT-23, F.Cu at (167.3, 126.5)
- added Q2: BC817, PCM_Package_TO_SOT_SMD_AKL:SOT-23, F.Cu at (166.5, 69.2)
- added Q3: BC817, PCM_Package_TO_SOT_SMD_AKL:SOT-23, F.Cu at (198.3, 69.0)
- added Q4: BC817, PCM_Package_TO_SOT_SMD_AKL:SOT-23, F.Cu at (159.5, 69.2)
- added Q5: BC817, PCM_Package_TO_SOT_SMD_AKL:SOT-23, F.Cu at (221.0, 127.5)
- added Q6: BC817, PCM_Package_TO_SOT_SMD_AKL:SOT-23, F.Cu at (188.2, 68.8)
- added Q7: BC817, PCM_Package_TO_SOT_SMD_AKL:SOT-23, F.Cu at (182.8, 114.4)
- added Q8: BC817, PCM_Package_TO_SOT_SMD_AKL:SOT-23, F.Cu at (193.0, 114.4)
- added Q9: BC817, PCM_Package_TO_SOT_SMD_AKL:SOT-23, F.Cu at (217.2, 127.5)
- added R17: 470k, PCM_Resistor_SMD_AKL:R_0603_1608Metric, F.Cu at (99.7, 100.1)
- added R18: 15, PCM_Resistor_SMD_AKL:R_0603_1608Metric, F.Cu at (99.7, 102.9)
- added R19: 10K, PCM_Resistor_SMD_AKL:R_0603_1608Metric, F.Cu at (171.6, 68.0)
- added R20: 10K, PCM_Resistor_SMD_AKL:R_0603_1608Metric, F.Cu at (171.6, 78.7)
- added R21: 10K, PCM_Resistor_SMD_AKL:R_0603_1608Metric, F.Cu at (163.0, 68.2)
- added R22: 2.4K, PCM_Resistor_SMD_AKL:R_0603_1608Metric, F.Cu at (166.8, 72.0)
- added R23: 4.7K, PCM_Resistor_SMD_AKL:R_0603_1608Metric, F.Cu at (203.4, 68.0)
- added R24: 2.4K, PCM_Resistor_SMD_AKL:R_0603_1608Metric, F.Cu at (203.6, 78.8)
- added R25: 10K, PCM_Resistor_SMD_AKL:R_0603_1608Metric, F.Cu at (194.6, 68.0)
- added R26: 47K, PCM_Resistor_SMD_AKL:R_0603_1608Metric, F.Cu at (194.5, 70.0)
- added R27: 2.4K, PCM_Resistor_SMD_AKL:R_0603_1608Metric, F.Cu at (198.5, 72.0)
- added R28: 10K, PCM_Resistor_SMD_AKL:R_0603_1608Metric, F.Cu at (156.0, 68.2)
- added R29: 2.4K, PCM_Resistor_SMD_AKL:R_0603_1608Metric, F.Cu at (159.8, 72.0)
- added R30: 2.4k, PCM_Resistor_SMD_AKL:R_0603_1608Metric, F.Cu at (223.8, 125.4)
- added R31: 10k, PCM_Resistor_SMD_AKL:R_0603_1608Metric, F.Cu at (221.3, 124.6)
- added R32: 10K, PCM_Resistor_SMD_AKL:R_0603_1608Metric, F.Cu at (184.6, 67.8)
- added R33: 47K, PCM_Resistor_SMD_AKL:R_0603_1608Metric, F.Cu at (184.6, 69.5)
- added R34: 2.4K, PCM_Resistor_SMD_AKL:R_0603_1608Metric, F.Cu at (188.4, 71.5)
- added R35: 2.4k, PCM_Resistor_SMD_AKL:R_0603_1608Metric, F.Cu at (183.0, 111.5)
- added R36: 2.4k, PCM_Resistor_SMD_AKL:R_0603_1608Metric, F.Cu at (193.3, 111.5)
- added R37: 2.4k, PCM_Resistor_SMD_AKL:R_0603_1608Metric, F.Cu at (214.9, 124.6)
- added R38: 10k, PCM_Resistor_SMD_AKL:R_0603_1608Metric, F.Cu at (214.2, 127.2)
- added R39: 2.4k, PCM_Resistor_SMD_AKL:R_0603_1608Metric, F.Cu at (164.6, 114.8)
- added R40: 10k, PCM_Resistor_SMD_AKL:R_0603_1608Metric, F.Cu at (165.5, 117.6)
- added R41: 4.7k, PCM_Resistor_SMD_AKL:R_0603_1608Metric, F.Cu at (162.7, 120.5)
- added R42: 10k, PCM_Resistor_SMD_AKL:R_0603_1608Metric, F.Cu at (159.2, 120.6)
- added R43: 10k, PCM_Resistor_SMD_AKL:R_0603_1608Metric, F.Cu at (158.6, 127.6)
- added R44: 2.4k, PCM_Resistor_SMD_AKL:R_0603_1608Metric, F.Cu at (154.6, 115.2)
- added R45: 10k, PCM_Resistor_SMD_AKL:R_0603_1608Metric, F.Cu at (151.2, 117.7)
- added R46: 4.7k, PCM_Resistor_SMD_AKL:R_0603_1608Metric, F.Cu at (147.0, 127.4)
- added R47: 10k, PCM_Resistor_SMD_AKL:R_0603_1608Metric, F.Cu at (154.2, 121.0)
- added R48: 10k, PCM_Resistor_SMD_AKL:R_0603_1608Metric, F.Cu at (150.3, 127.3)
- added R49: 2.4k, PCM_Resistor_SMD_AKL:R_0603_1608Metric, F.Cu at (173.5, 115.2)
- added R50: 10k, PCM_Resistor_SMD_AKL:R_0603_1608Metric, F.Cu at (174.2, 117.6)
- added R51: 4.7k, PCM_Resistor_SMD_AKL:R_0603_1608Metric, F.Cu at (171.5, 120.9)
- added R52: 10k, PCM_Resistor_SMD_AKL:R_0603_1608Metric, F.Cu at (167.7, 122.4)
- added R53: 10k, PCM_Resistor_SMD_AKL:R_0603_1608Metric, F.Cu at (174.6, 127.6)
- added R54: 2.5k, PCM_Resistor_SMD_AKL:R_0603_1608Metric, F.Cu at (93.6, 97.4)
- added R55: 470k, PCM_Resistor_SMD_AKL:R_0603_1608Metric, F.Cu at (93.6, 100.1)
- added R56: 15, PCM_Resistor_SMD_AKL:R_0603_1608Metric, F.Cu at (93.6, 102.9)
- added R57: 1k, PCM_SparkFun-Resistor:R_0603_1608Metric, F.Cu at (135.9, 64.5)
- added U4: ~, Lib_GP8211S-TC50-EW:ESOP-8_L4.9-W3.9-P1.27-LS6.0-BL-EP, F.Cu at (207.4, 120.8)
- added U5: ~, Package_SO:SSOP-10-1EP_3.9x4.9mm_P1mm_EP2.1x3.3mm, F.Cu at (47.2, 101.0)
- added U6: ~, Package_SO:SSOP-10-1EP_3.9x4.9mm_P1mm_EP2.1x3.3mm, F.Cu at (47.2, 85.0)
- added U7: AP63203WU, Package_TO_SOT_SMD:TSOT-23-6, F.Cu at (142.1, 74.0)
- added U8: ESP32-S3-MINI-1U, RF_Module:ESP32-S2-MINI-1U, F.Cu at (219.8, 97.3)
- D1: value SM712 -> TVA; footprint PCM_Package_TO_SOT_SMD_AKL:SOT-23 -> PCM_Diode_SMD_AKL:D_SOD-123F
- J1: value NPN_IN -> Screw_Terminal_9_P3.50mm; footprint TerminalBlock_Phoenix:TerminalBlock_Phoenix_PT-1,5-4-3.5-H_1x04_P3.50mm_Horizontal -> TerminalBlock_Phoenix:TerminalBlock_Phoenix_PT-1,5-9-5.0-H_1x09_P5.00mm_Horizontal
- J2: value PNP_IN -> Screw_Terminal_9_P5.00mm; footprint TerminalBlock_Phoenix:TerminalBlock_Phoenix_PT-1,5-4-3.5-H_1x04_P3.50mm_Horizontal -> TerminalBlock_Phoenix:TerminalBlock_Phoenix_PT-1,5-9-5.0-H_1x09_P5.00mm_Horizontal
- J3: value RS485 -> Screw_Terminal_9_P5.00mm; footprint TerminalBlock_Phoenix:TerminalBlock_Phoenix_PT-1,5-3-3.5-H_1x03_P3.50mm_Horizontal -> TerminalBlock_Phoenix:TerminalBlock_Phoenix_PT-1,5-9-5.0-H_1x09_P5.00mm_Horizontal
- J4: value NPN_Out -> Screw_Terminal_9_P5.00mm; footprint TerminalBlock_Phoenix:TerminalBlock_Phoenix_PT-1,5-4-3.5-H_1x04_P3.50mm_Horizontal -> TerminalBlock_Phoenix:TerminalBlock_Phoenix_PT-1,5-9-5.0-H_1x09_P5.00mm_Horizontal
- OC1, OC2, OC3, OC4: value FOD817S -> TLP293; footprint PCM_Package_DIP_AKL:SMDIP-4_W9.53mm -> PCM_Package_SO_AKL:SOP-4_4.4x2.6mm_P1.27mm
- R1, R2, R3, R4, R5: value 2.4K -> 10k
- R10, R11: value 2.4K -> 470; footprint PCM_Resistor_SMD_AKL:R_0603_1608Metric -> PCM_SparkFun-Resistor:R_0603_1608Metric
- R12: value 2.4K -> 20K
- R13, R6, R7: value 2.4K -> 10K
- R14, R15: value 2.4K -> 4.7k
- R16: value 2.4K -> 2.5k
- R8: value 2.4K -> 4.7K
- U1: value ESP32-S3-WROOM-1 -> SP3485EN; footprint RF_Module:ESP32-S3-WROOM-1 -> Package_SO:SOIC-8_3.9x4.9mm_P1.27mm
- moved J2 214.2 mm to (227.0, 62.3), turned to 180 degrees
- moved J4 168.5 mm to (187.0, 134.3)
- moved J1 167.1 mm to (180.9, 62.2), turned to 180 degrees
- moved R9 162.3 mm to (208.6, 78.8), turned to 180 degrees
- moved R15 159.1 mm to (207.8, 115.5), turned to -90 degrees
- moved OC2 143.1 mm to (208.6, 73.4), turned to -90 degrees
- moved OC4 141.6 mm to (203.4, 73.5), turned to -90 degrees
- moved R8 139.4 mm to (208.6, 68.0)
- moved D1 136.0 mm to (208.2, 128.0)
- moved R14 130.7 mm to (209.6, 115.5), turned to -90 degrees
- moved U1 118.9 mm to (158.0, 102.2)
- moved R12 114.7 mm to (180.7, 70.5), turned to -90 degrees
- moved J3 110.5 mm to (140.9, 134.2)
- moved R7 108.3 mm to (176.3, 78.6)
- moved R6 107.4 mm to (176.3, 68.0)
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Connections:
- D1 pad 1: /Board-PLC4UNI-G1W/con_RS485_B -> /Board-PLC4UNI-G1W/Out_0-10V
- D1 pad 2: /Board-PLC4UNI-G1W/con_RS485_A -> GND
- J1 pad 1: /Board-PLC4UNI-G1W/IN_NPN1 -> /Board-PLC4UNI-G1W/IN_0-10V
- J1 pad 2: /Board-PLC4UNI-G1W/IN_NPN2 -> /Board-PLC4UNI-G1W/IN_NPN2_Opto
- J1 pad 3: /Board-PLC4UNI-G1W/IN_NPN3 -> /Board-PLC4UNI-G1W/IN_NPN1_Opto
- J1 pad 4: /Board-PLC4UNI-G1W/IN_NPN4 -> /Board-PLC4UNI-G1W/IN_NPN2
- J2 pad 1: /Board-PLC4UNI-G1W/IN_PNP1 -> /IN_CT2
- J2 pad 2: /Board-PLC4UNI-G1W/IN_PNP2 -> /IN_CT1
- J2 pad 3: /Board-PLC4UNI-G1W/IN_PNP3 -> /IN_VAC2
- J2 pad 4: /Board-PLC4UNI-G1W/IN_PNP4 -> /IN_VAC1
- J3 pad 3: GNDPWR -> GND
- J4 pad 1: unconnected-(J4-Pad1) -> /Board-PLC4UNI-G1W/out-no-2
- J4 pad 2: unconnected-(J4-Pad2) -> /Board-PLC4UNI-G1W/out-common-2
- J4 pad 3: unconnected-(J4-Pad3) -> /Board-PLC4UNI-G1W/Out_4-20mA
- J4 pad 4: unconnected-(J4-Pad4) -> /Out_4-20mA_2
- OC1 pad 2: /Board-PLC4UNI-G1W/IN_NPN3 -> /Board-PLC4UNI-G1W/IN_NPN2_Opto
- OC1 pad 4: /Board-PLC4UNI-G1W/Input_NPN3/Out -> /Board-PLC4UNI-G1W/Input_NPN1_Opto1/OUT
- OC2 pad 2: /Board-PLC4UNI-G1W/IN_NPN1 -> GND
- OC2 pad 4: /Board-PLC4UNI-G1W/Input_NPN1/Out -> /Board-PLC4UNI-G1W/Input_PNP2_Opto/OUT
- OC3 pad 2: /Board-PLC4UNI-G1W/IN_NPN2 -> /Board-PLC4UNI-G1W/IN_NPN1_Opto
- OC3 pad 4: /Board-PLC4UNI-G1W/Input_NPN2/Out -> /Board-PLC4UNI-G1W/Input_NPN1_Opto/OUT
- OC4 pad 4: /Board-PLC4UNI-G1W/Input_PNP3/Out -> /Board-PLC4UNI-G1W/Input_PNP1_Opto/OUT
- R1 pad 1: Net-(OC2-Pad1) -> /Board-PLC4UNI-G1W/con_RS485_A
- R1 pad 2: VCC -> +3.3V
- R10 pad 1: /Board-PLC4UNI-G1W/Input_PNP2/Out -> Net-(R10-Pad1)
- R10 pad 2: +3.3V -> /Board-PLC4UNI-G1W/Output_NPN_Opto1/IN
- R11 pad 1: Net-(OC3-Pad1) -> Net-(R11-Pad1)
- R11 pad 2: VCC -> /Board-PLC4UNI-G1W/Output_NPN_Opto/IN
- R12 pad 1: Net-(OC1-Pad1) -> /Board-PLC4UNI-G1W/IN_0-10V
- R12 pad 2: VCC -> /Board-PLC4UNI-G1W/Input_0-10V/ADC_IN_3V3
- R13 pad 1: Net-(OC7-Pad1) -> /Board-PLC4UNI-G1W/Input_0-10V/ADC_IN_3V3
- R13 pad 2: VCC -> GND
- R14 pad 1: /Board-PLC4UNI-G1W/Input_NPN4/Out -> +3.3V
- R14 pad 2: +3.3V -> /Board-PLC4UNI-G1W/Output_0-10V/SCL
- R15 pad 1: /Board-PLC4UNI-G1W/IN_PNP4 -> +3.3V
- R15 pad 2: Net-(OC8-Pad1) -> /Board-PLC4UNI-G1W/Output_0-10V/SDA
- R16 pad 1: /Board-PLC4UNI-G1W/Input_PNP4/Out -> Net-(U5-SET)
- R16 pad 2: +3.3V -> GND
- R2 pad 1: /Board-PLC4UNI-G1W/IN_PNP3 -> /Board-PLC4UNI-G1W/con_RS485_B
- R2 pad 2: Net-(OC4-Pad1) -> /Board-PLC4UNI-G1W/con_RS485_A
- R3 pad 1: /Board-PLC4UNI-G1W/Input_PNP3/Out -> GND
- R3 pad 2: +3.3V -> /Board-PLC4UNI-G1W/con_RS485_B
- R4 pad 1: /Board-PLC4UNI-G1W/Input_NPN3/Out -> +3.3V
- R4 pad 2: +3.3V -> /Board-PLC4UNI-G1W/Output_0-10V/SCL
- R5 pad 1: /Board-PLC4UNI-G1W/Input_NPN1/Out -> +3.3V
- R5 pad 2: +3.3V -> /Board-PLC4UNI-G1W/Output_0-10V/SDA
- R6 pad 1: /Board-PLC4UNI-G1W/Input_NPN2/Out -> VCC
- R6 pad 2: +3.3V -> Net-(OC1-Pad1)
- R7 pad 1: /Board-PLC4UNI-G1W/IN_PNP1 -> +3.3V
- R7 pad 2: Net-(OC5-Pad1) -> /Board-PLC4UNI-G1W/Input_NPN1_Opto1/OUT
- R8 pad 1: /Board-PLC4UNI-G1W/Input_PNP1/Out -> /Board-PLC4UNI-G1W/IN_PNP2_Opto
- R8 pad 2: +3.3V -> Net-(OC2-Pad1)
- R9 pad 1: /Board-PLC4UNI-G1W/IN_PNP2 -> /Board-PLC4UNI-G1W/Input_PNP2_Opto/OUT
- R9 pad 2: Net-(OC6-Pad1) -> +3.3V
- U1 pad 1: GND -> /Board-PLC4UNI-G1W/PLC4UNI/micro_rs485_tx
- U1 pad 2: +3.3V -> /Board-PLC4UNI-G1W/RS485_Module1_protect/~{TX}/RX
- U1 pad 3: unconnected-(U1-EN-Pad3) -> /Board-PLC4UNI-G1W/RS485_Module1_protect/~{TX}/RX
- U1 pad 4: unconnected-(U1-IO4-Pad4) -> /Board-PLC4UNI-G1W/PLC4UNI/micro_rs485_rx
- U1 pad 5: unconnected-(U1-IO5-Pad5) -> GND
- U1 pad 6: unconnected-(U1-IO6-Pad6) -> /Board-PLC4UNI-G1W/con_RS485_A
- U1 pad 7: unconnected-(U1-IO7-Pad7) -> /Board-PLC4UNI-G1W/con_RS485_B
- U1 pad 8: unconnected-(U1-IO15-Pad8) -> +3.3V
Routing:
- net GND: track 0.00 -> 163.6 mm, vias 0 -> 16
- net +3.3V: track 0.00 -> 114.5 mm
- net VCC: track 0.00 -> 47.7 mm
- net /Board-PLC4UNI-G1W/out-no-2: track 0.00 -> 21.7 mm
- net /Board-PLC4UNI-G1W/out-no-1: track 0.00 -> 20.6 mm
- net /Board-PLC4UNI-G1W/out-nc: track 0.00 -> 20.4 mm
- net Net-(D6-A): track 0.00 -> 17.4 mm
- net Net-(D5-A): track 0.00 -> 17.2 mm
- net Net-(Q12-C): track 0.00 -> 16.1 mm
- net /Board-PLC4UNI-G1W/PNP_OUT3: track 0.00 -> 16.1 mm
- net /Board-PLC4UNI-G1W/out-common-1: track 0.00 -> 15.1 mm
- net /Board-PLC4UNI-G1W/PNP_OUT2: track 0.00 -> 13.9 mm
- net /Board-PLC4UNI-G1W/PNP_OUT1: track 0.00 -> 13.7 mm
- net /Board-PLC4UNI-G1W/out-common-2: track 0.00 -> 12.0 mm
- net Net-(Q12-B): track 0.00 -> 11.3 mm
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- added copper zone on F.Cu, net +3.3V
- added copper zone on F.Cu, net GND
- added copper zone on In1.Cu, net GND
- added copper zone on F.Cu, net Net-(U7-SW)
Other:
- board outline added: 100 x 80.2 mm
- copper layers 2 -> 4

Commit message: Add files via upload
Parts:
- removed R10, R11: 470, PCM_SparkFun-Resistor:R_0603_1608Metric
- removed R4, R5: 10k, PCM_Resistor_SMD_AKL:R_0603_1608Metric
- added J6: PINHD_2x5_Male, Connector_PinHeader_2.54mm:PinHeader_2x05_P2.54mm_Horizontal, F.Cu at (146.6, 103.4)
- moved C6 191.8 mm to (231.5, 118.6), turned to 180 degrees
- moved C5 189.0 mm to (228.0, 121.8), turned to 180 degrees
- moved C7 187.3 mm to (227.6, 108.3)
- moved U5 183.5 mm to (230.3, 113.6), turned to -90 degrees
- moved D3 179.2 mm to (227.5, 126.8), turned to 90 degrees
- moved D2 177.9 mm to (226.6, 111.6), turned to -90 degrees
- moved C10 166.6 mm to (206.4, 103.0), turned to 180 degrees
- moved C9 165.0 mm to (203.5, 111.2), turned to 90 degrees
- moved U6 163.4 mm to (208.8, 110.0), turned to 180 degrees
- moved D10 162.4 mm to (210.5, 106.2), turned to 180 degrees
- moved C8 161.9 mm to (200.5, 107.5), turned to 90 degrees
- moved D11 151.8 mm to (199.8, 111.8), turned to -90 degrees
- moved R17 133.1 mm to (230.2, 125.8)
- moved R18 132.9 mm to (230.2, 127.8), turned to 180 degrees
- moved R16 130.2 mm to (228.2, 118.6), turned to 180 degrees
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Connections:
- U8 pad 12: unconnected-(U8-IO8-Pad12) -> /Board-PLC4UNI-G1W/Output_0-10V/SDA
- U8 pad 13: unconnected-(U8-IO9-Pad13) -> /Board-PLC4UNI-G1W/Output_0-10V/SCL
- U8 pad 23: unconnected-(U8-USB_D--Pad23) -> /Board-PLC4UNI-G1W/PLC4UNI/USB-
- U8 pad 24: unconnected-(U8-USB_D+-Pad24) -> /Board-PLC4UNI-G1W/PLC4UNI/USB+
- U8 pad 25: unconnected-(U8-IO21-Pad25) -> /Board-PLC4UNI-G1W/Input_NPN1/OUT
- U8 pad 26: unconnected-(U8-IO26-Pad26) -> /Board-PLC4UNI-G1W/Input_NPN/OUT
- U8 pad 27: unconnected-(U8-IO47-Pad27) -> /Board-PLC4UNI-G1W/Output_NPN_Opto1/IN
- U8 pad 28: unconnected-(U8-IO33-Pad28) -> /Board-PLC4UNI-G1W/Input_PNP1_Opto/OUT
- U8 pad 29: unconnected-(U8-IO34-Pad29) -> /Board-PLC4UNI-G1W/Input_PNP2_Opto/OUT
- U8 pad 30: unconnected-(U8-IO48-Pad30) -> /Board-PLC4UNI-G1W/OutputRelay1/IN
- U8 pad 31: unconnected-(U8-IO35-Pad31) -> /Board-PLC4UNI-G1W/Input_NPN1_Opto/OUT
- U8 pad 32: unconnected-(U8-IO36-Pad32) -> /Board-PLC4UNI-G1W/Input_NPN1_Opto1/OUT
- U8 pad 33: unconnected-(U8-IO37-Pad33) -> /Board-PLC4UNI-G1W/Input_PNP/OUT
- U8 pad 34: unconnected-(U8-IO38-Pad34) -> /Board-PLC4UNI-G1W/Input_PNP2/OUT
- U8 pad 35: unconnected-(U8-IO39-Pad35) -> /Board-PLC4UNI-G1W/PLC4UNI/Out_4-20mA
- U8 pad 36: unconnected-(U8-IO40-Pad36) -> /Board-PLC4UNI-G1W/PLC4UNI/Out_4-20mA_2
- U8 pad 37: unconnected-(U8-IO41-Pad37) -> /Board-PLC4UNI-G1W/Output_PNP/IN
- U8 pad 38: unconnected-(U8-IO42-Pad38) -> /Board-PLC4UNI-G1W/Output_PNP1/IN
- U8 pad 4: unconnected-(U8-IO0-Pad4) -> /Board-PLC4UNI-G1W/Output_NPN1/IN
- U8 pad 41: unconnected-(U8-IO45-Pad41) -> /Board-PLC4UNI-G1W/Output_PNP2/IN
- U8 pad 44: unconnected-(U8-IO46-Pad44) -> /Board-PLC4UNI-G1W/Output_NPN_Opto/IN
- U8 pad 5: unconnected-(U8-IO1-Pad5) -> /Board-PLC4UNI-G1W/Output_NPN/IN
- U8 pad 6: unconnected-(U8-IO2-Pad6) -> /Board-PLC4UNI-G1W/OutRelay2/IN
- U8 pad 7: unconnected-(U8-IO3-Pad7) -> /Board-PLC4UNI-G1W/PLC4UNI/IN_4-20mA
- U8 pad 8: unconnected-(U8-IO4-Pad8) -> /Board-PLC4UNI-G1W/PLC4UNI/IN_4-20mA_2
- U8 pad 9: unconnected-(U8-IO5-Pad9) -> /Board-PLC4UNI-G1W/PLC4UNI/micro1_rs485_control
Routing:
- net VCC: track 47.7 -> 272.5 mm, vias 0 -> 14
- net +3.3V: track 114.5 -> 298.7 mm, vias 0 -> 6
- net GND: track 163.6 -> 279.6 mm, vias 16 -> 28
- net /Board-PLC4UNI-G1W/PLC4UNI/micro_rs485_tx: track 0.00 -> 84.4 mm
- net /Board-PLC4UNI-G1W/PLC4UNI/micro_rs485_rx: track 0.00 -> 83.5 mm, vias 0 -> 2
- net /Board-PLC4UNI-G1W/Output_0-10V/SDA: track 1.76 -> 51.2 mm, vias 0 -> 2
- net /Board-PLC4UNI-G1W/con_RS485_B: track 0.00 -> 44.4 mm
- net /Board-PLC4UNI-G1W/Output_0-10V/SCL: track 1.74 -> 35.9 mm
- net /Board-PLC4UNI-G1W/con_RS485_A: track 0.00 -> 29.0 mm
- net Net-(D2-A): track 0.00 -> 24.6 mm
- net Net-(U6-SET): track 0.00 -> 5.84 mm
- net Net-(U5-SET): track 0.00 -> 5.76 mm
- net Net-(D10-A): track 0.00 -> 5.67 mm
- net Net-(D11-A1): track 0.00 -> 3.52 mm
- net Net-(U6-V5V): track 0.00 -> 2.67 mm
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